File: NeuMaE/NeuMaE.sch (KiCad schematic (older format))
At the start: 20 parts, among them J1 MOTOR, J2 PROGRAM, J3 LED, J4 PWR, J5 EXTRA, Q1 BC337, SW1 FLASH, SW2 RESET, U1 PMIC-LD1117V33(TO-220), U2 ESP8266-12E_ESP-12E

Commit message: made board smaller
Parts:
- added J6: PWR, Connector_PinHeader_2.54mm:PinHeader_1x02_P2.54mm_Vertical, symbol Connector:Conn_01x02_Male
Connections:
- net +3V3: now also J6.1 (Pin_1)
- net GND: now also J6.2 (Pin_2)
Changed lines of the file:
@@
 Wire Wire Line
 	3325 3400 3125 3400
+$Comp
+L Connector:Conn_01x02_Male J6
+U 1 1 5E6026BD
+P 2025 2450
+F 0 "J6" H 2131 2628 50  0000 C CNN
+F 1 "PWR" H 2131 2537 50  0000 C CNN
+F 2 "Connector_PinHeader_2.54mm:PinHeader_1x02_P2.54mm_Vertical" H 2025 2450 50  0001 C CNN
+F 3 "~" H 2025 2450 50  0001 C CNN
+	1    2025 2450
+	1    0    0    -1
+$EndComp
+$Comp
+L power:+3V3 #PWR0118
+U 1 1 5E6035E1
+P 2225 2450
+F 0 "#PWR0118" H 2225 2300 50  0001 C CNN
+F 1 "+3V3" V 2240 2578 50  0000 L CNN
+F 2 "" H 2225 2450 50  0001 C CNN
+F 3 "" H 2225 2450 50  0001 C CNN
+	1    2225 2450
+	0    1    1    0
+$EndComp
+$Comp
+L power:GND #PWR0119
+U 1 1 5E6036C7
+P 2225 2550
+F 0 "#PWR0119" H 2225 2300 50  0001 C CNN
+F 1 "GND" H 2230 2377 50  0000 C CNN
+F 2 "" H 2225 2550 50  0001 C CNN
+F 3 "" H 2225 2550 50  0001 C CNN
+	1    2225 2550
+	1    0    0    -1
+$EndComp
 $EndSCHEMATC

Commit message: fixed C1 footprint
Parts:
- C1: footprint Capacitor_THT:C_Rect_L4.6mm_W2.0mm_P2.50mm_MKS02_FKP02 -> Capacitor_THT:C_Rect_L7.2mm_W2.5mm_P5.00mm_FKS2_FKP2_MKS2_MKP2
Changed lines of the file:
@@
 F 0 "C1" H 942 1096 50  0000 L CNN
 F 1 "100nF" H 942 1005 50  0000 L CNN
-F 2 "Capacitor_THT:C_Rect_L4.6mm_W2.0mm_P2.50mm_MKS02_FKP02" H 850 1050 50  0001 C CNN
+F 2 "Capacitor_THT:C_Rect_L7.2mm_W2.5mm_P5.00mm_FKS2_FKP2_MKS2_MKP2" H 850 1050 50  0001 C CNN
 F 3 "~" H 850 1050 50  0001 C CNN
 	1    850  1050

Commit message: added recoil diode
Parts:
- added D1: RECOIL, Diode_THT:D_DO-35_SOD27_P2.54mm_Vertical_AnodeUp, symbol Device:D_Schottky
Connections:
- net +3V3: now also D1.1 (K)
- net at J1.1 (Pin_1), Q1.1 (C): now also D1.2 (A)
Other:
- moved on the sheet: J1, J4, J6, Q1, R2, R3, R7, R8
